Commit message: mar4

File: assets/urdf/xarm.urdf (robot description, URDF)
Before this commit: robot xarm, 13 links, 12 joints
Links:
- added link camera_link; visual sphere radius=0.01
Joints:
- added joint camera_joint: type fixed, parent hand_link, child camera_link, origin xyz=-0.025 0 0.05 rpy=0 0 0
